File: kicad/a2pdp11.kicad_pcb (KiCad board)
At the start: 2 copper layers, 196.9 x 77.5 mm, 45 parts, among them J1 DCJ11A, J2 DCJ11B, J3 TN9A, J4 TN9A, J5 A2BUSA, J6 A2BUSB, J7 3V3, J8 5V, J9 Jumper, SW1 HALT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

Commit message: Apple II Interface
Parts:
- removed A1BUS1: A2_BUS, Apple2_bus:BUS_A2
- removed J10: ~, Connector_PinSocket_2.54mm:PinSocket_2x03_P2.54mm_Vertical
- added A2BUS1: A2_BUS, Apple2_bus:BUS_A2, F.Cu at (210.2, 130.8)
- moved J5 1.27 mm to (248.3, 119.4)
Connections:
- J1 pad 19: /MAP -> Net-(J1-Pin_19)
- J1 pad 2: /AIO0 -> Net-(J1-Pin_2)
- J1 pad 3: /AIO1 -> Net-(J1-Pin_3)
- J1 pad 4: /AIO2 -> Net-(J1-Pin_4)
- J1 pad 5: /AIO3 -> Net-(J1-Pin_5)
- J4 pad 2: /A3 -> /AIO0
- J4 pad 3: /A2 -> /AIO1
- J4 pad 4: /A1 -> /AIO2
- J4 pad 5: /A0 -> /AIO3
- J5 pad 16: Net-(A1BUS1-~{DEVSEL}) -> Net-(A2BUS1-~{DEVSEL})
- J6 pad 17: Net-(A1BUS1-A7) -> /A7
- J6 pad 18: Net-(A1BUS1-A6) -> /A6
- J6 pad 19: Net-(A1BUS1-A5) -> /A5
- J6 pad 20: Net-(A1BUS1-A4) -> /A4
- J6 pad 21: Net-(A1BUS1-A3) -> /A3
- J6 pad 22: Net-(A1BUS1-A2) -> /A2
- J6 pad 23: Net-(A1BUS1-A1) -> /A1
- J6 pad 24: Net-(A1BUS1-A0) -> /A0
- J6 pad 25: Net-(A1BUS1-~{I/O_SEL}) -> Net-(A2BUS1-~{I/O_SEL})
- JP2 pad 2: Net-(A1BUS1-~{I/O_SEL}) -> Net-(A2BUS1-~{DEVSEL})
- U1 pad 19: /MAP -> Net-(J1-Pin_19)
- U1 pad 2: /AIO0 -> Net-(J1-Pin_2)
- U1 pad 3: /AIO1 -> Net-(J1-Pin_3)
- U1 pad 4: /AIO2 -> Net-(J1-Pin_4)
- U1 pad 5: /AIO3 -> Net-(J1-Pin_5)
- U11 pad 2: Net-(A1BUS1-~{DEVSEL}) -> Net-(A2BUS1-~{I/O_SEL})
- U5 pad 11: Net-(J10-Pin_6) -> /DAL5
- U5 pad 12: Net-(J10-Pin_4) -> /DAL4
- U5 pad 13: Net-(J10-Pin_2) -> /DAL3
- U5 pad 2: /AIO0 -> /A7
- U5 pad 3: /AIO1 -> /A6
- U5 pad 4: /AIO2 -> /A5
- U5 pad 5: /AIO3 -> /A4
- U5 pad 6: /MAP -> /A3
- U5 pad 7: Net-(J10-Pin_1) -> /A2
- U5 pad 8: Net-(J10-Pin_3) -> /A1
- U5 pad 9: Net-(J10-Pin_5) -> /A0
- U6 pad 11: /A3 -> /AIO0
- U6 pad 12: /A2 -> /AIO1
- U6 pad 13: /A1 -> /AIO2
- U6 pad 14: /A0 -> /AIO3
- U6 pad 6: Net-(A1BUS1-A0) -> Net-(J1-Pin_5)
- U6 pad 7: Net-(A1BUS1-A1) -> Net-(J1-Pin_4)
- U6 pad 8: Net-(A1BUS1-A2) -> Net-(J1-Pin_3)
- U6 pad 9: Net-(A1BUS1-A3) -> Net-(J1-Pin_2)
- U8 pad 44: /A0 -> /AIO3
- U8 pad 45: /A1 -> /AIO2
- U8 pad 46: /A2 -> /AIO1
- U8 pad 47: /A3 -> /AIO0
Routing:
- net /A7: track 0.00 -> 153.8 mm
- net /A6: track 0.00 -> 148.3 mm
- net /A5: track 0.00 -> 142.3 mm
- net /A4: track 0.00 -> 130.1 mm
- net /AIO1: track 16.3 -> 128.7 mm
- net /AIO0: track 16.3 -> 128.5 mm
- net /AIO2: track 16.3 -> 128.3 mm
- net /AIO3: track 16.3 -> 127.9 mm
- net Net-(J1-Pin_2): track 0.00 -> 111.2 mm, vias 0 -> 1
- net Net-(J1-Pin_3): track 0.00 -> 106.4 mm, vias 0 -> 1
- net Net-(J1-Pin_4): track 0.00 -> 102.3 mm, vias 0 -> 1
- net Net-(J1-Pin_5): track 0.00 -> 98.4 mm, vias 0 -> 1
- net Net-(A1BUS1-A3): track 97.0 -> 0.00 mm
- net Net-(A1BUS1-A2): track 96.3 -> 0.00 mm
- net Net-(A1BUS1-A1): track 95.5 -> 0.00 mm
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
Commit message: Change I/O signal to IOSEL
Parts:
- JP2: value IOSEL-HALT -> DEVSEL-HALT
Connections:
- J1 pad 10: /IRQ1 -> /IRQ0
- J1 pad 11: /IRQ0 -> /IRQ1
- J4 pad 19: /IRQ0 -> /IRQ1
- J4 pad 20: /IRQ1 -> /IRQ0
- U1 pad 10: /IRQ1 -> /IRQ0
- U1 pad 11: /IRQ0 -> /IRQ1
- U8 pad 29: /IRQ1 -> /IRQ0
- U8 pad 30: /IRQ0 -> /IRQ1
Routing:
- net /IRQ1: track 115.6 -> 117.2 mm
- net /IRQ0: track 117.2 -> 115.6 mm
- net Net-(A2BUS1-~{I/O_SEL}): track 51.7 -> 50.7 mm
- net GND: vias 122 -> 127
Other:
- board text added: "Apple II PDP11 Card v0.17 2024 nanja.info"
- board text removed: "Apple II PDP11 Card v0.15 2024 nanja.info"
